Commit message: Add Can.stl in robot

File: robot_ws/src/bumblebee_description/urdf/bumblebee.urdf.xacro (robot description, xacro)
@@ -14,4 +14,17 @@
         <child link="base_link" />
         <origin rpy="0 0 0" xyz="0 0 0.033" />
+    </joint>
+    <link name="can_link">
+        <visual>
+            <origin rpy="1.57 0 0" xyz="-0.03 0.03 0" />
+            <geometry>
+                <mesh filename="package://bumblebee_description/meshes/can.STL" />
+            </geometry>
+        </visual>
+    </link>
+    <joint name="can_joint" type="fixed">
+        <parent link="base_link" />
+        <child link="can_link" />
+        <origin rpy="0 0 0" xyz="0 0 0.078" />
     </joint>
     <link name="wheel_left_link">
